File: ISA_ES688.sch (KiCad schematic (older format))
At the start: 108 parts, among them J1 LINE IN, J11 ISA BUS, J2 LINE OUT, J3 Joystick/MIDI, J4 Interrupt Select, J5 Address Select, J6 DMA Select, J7 SPKR OUT, J8 MIC, U1 L78L05, U2 74LS14, U3 ES688F, U4 74LS245, U5 74LS244, U6 NE558, U7 LM1877, U7 YMF262-M, U8 YAC512, U9 LM3403, Y1 14.318Mhz

Commit message: Assign more footprints
Parts:
- C10, C13, C14, C15, C16, C17, C18, C19: renamed from C?; footprint Capacitor_THT:C_Disc_D6.0mm_W2.5mm_P5.00mm -> Capacitor_SMD:C_1206_3216Metric_Pad1.33x1.80mm_HandSolder
- C20: renamed from C4; footprint Capacitor_THT:C_Disc_D6.0mm_W2.5mm_P5.00mm -> Capacitor_SMD:C_1206_3216Metric_Pad1.33x1.80mm_HandSolder
- C21: renamed from C11; footprint Capacitor_THT:C_Disc_D6.0mm_W2.5mm_P5.00mm -> Capacitor_SMD:C_1206_3216Metric_Pad1.33x1.80mm_HandSolder
- C22: renamed from C8; footprint Capacitor_THT:C_Disc_D6.0mm_W2.5mm_P5.00mm -> Capacitor_SMD:C_1206_3216Metric_Pad1.33x1.80mm_HandSolder
- C23: renamed from C9; footprint Capacitor_THT:C_Disc_D6.0mm_W2.5mm_P5.00mm -> Capacitor_SMD:C_1206_3216Metric_Pad1.33x1.80mm_HandSolder
- C24: renamed from C5; footprint Capacitor_THT:C_Disc_D6.0mm_W2.5mm_P5.00mm -> Capacitor_SMD:C_1206_3216Metric_Pad1.33x1.80mm_HandSolder
- C25: renamed from C22; footprint Capacitor_THT:C_Disc_D6.0mm_W2.5mm_P5.00mm -> Capacitor_SMD:C_1206_3216Metric_Pad1.33x1.80mm_HandSolder
- C26, C28: renamed from C27; footprint Capacitor_THT:C_Disc_D6.0mm_W2.5mm_P5.00mm -> Capacitor_SMD:C_1206_3216Metric_Pad1.33x1.80mm_HandSolder
- C27, C53: renamed from C28; footprint Capacitor_THT:C_Disc_D6.0mm_W2.5mm_P5.00mm -> Capacitor_SMD:C_1206_3216Metric_Pad1.33x1.80mm_HandSolder
- C29: renamed from C24; footprint Capacitor_THT:C_Disc_D6.0mm_W2.5mm_P5.00mm -> Capacitor_SMD:C_1206_3216Metric_Pad1.33x1.80mm_HandSolder
- C3: renamed from C53; footprint Capacitor_THT:C_Disc_D6.0mm_W2.5mm_P5.00mm -> Capacitor_SMD:C_1206_3216Metric_Pad1.33x1.80mm_HandSolder
- C30: renamed from C6; footprint Capacitor_THT:C_Disc_D6.0mm_W2.5mm_P5.00mm -> Capacitor_SMD:C_1206_3216Metric_Pad1.33x1.80mm_HandSolder
- C31: renamed from C33; footprint Capacitor_THT:C_Disc_D6.0mm_W2.5mm_P5.00mm -> Capacitor_SMD:C_1206_3216Metric_Pad1.33x1.80mm_HandSolder
- C32: renamed from C10; footprint Capacitor_THT:C_Disc_D6.0mm_W2.5mm_P5.00mm -> Capacitor_SMD:C_1206_3216Metric_Pad1.33x1.80mm_HandSolder
- C36: renamed from C7; footprint Capacitor_THT:C_Disc_D6.0mm_W2.5mm_P5.00mm -> Capacitor_SMD:C_1206_3216Metric_Pad1.33x1.80mm_HandSolder
- C39: renamed from C47; footprint Capacitor_THT:C_Disc_D6.0mm_W2.5mm_P5.00mm -> Capacitor_SMD:C_1206_3216Metric_Pad1.33x1.80mm_HandSolder
- C40: renamed from C48; footprint Capacitor_THT:C_Disc_D6.0mm_W2.5mm_P5.00mm -> Capacitor_SMD:C_1206_3216Metric_Pad1.33x1.80mm_HandSolder
- C43: renamed from C38; footprint Capacitor_THT:C_Disc_D6.0mm_W2.5mm_P5.00mm -> Capacitor_SMD:C_1206_3216Metric_Pad1.33x1.80mm_HandSolder
- C44: renamed from C39; footprint Capacitor_THT:C_Disc_D6.0mm_W2.5mm_P5.00mm -> Capacitor_SMD:C_1206_3216Metric_Pad1.33x1.80mm_HandSolder
- C45: renamed from C31; footprint Capacitor_THT:C_Disc_D6.0mm_W2.5mm_P5.00mm -> Capacitor_SMD:C_1206_3216Metric_Pad1.33x1.80mm_HandSolder
- C46: renamed from C29; footprint Capacitor_THT:C_Disc_D6.0mm_W2.5mm_P5.00mm -> Capacitor_SMD:C_1206_3216Metric_Pad1.33x1.80mm_HandSolder
- C47: renamed from C26; footprint Capacitor_THT:C_Disc_D6.0mm_W2.5mm_P5.00mm -> Capacitor_SMD:C_1206_3216Metric_Pad1.33x1.80mm_HandSolder
- C48: renamed from C41; footprint Capacitor_THT:C_Disc_D6.0mm_W2.5mm_P5.00mm -> Capacitor_SMD:C_1206_3216Metric_Pad1.33x1.80mm_HandSolder
- C49: renamed from C40; footprint Capacitor_THT:C_Disc_D6.0mm_W2.5mm_P5.00mm -> Capacitor_SMD:C_1206_3216Metric_Pad1.33x1.80mm_HandSolder
- C5: renamed from C1; footprint Capacitor_THT:C_Disc_D6.0mm_W2.5mm_P5.00mm -> Capacitor_SMD:C_1206_3216Metric_Pad1.33x1.80mm_HandSolder
- C52: renamed from C30; footprint Capacitor_THT:C_Disc_D6.0mm_W2.5mm_P5.00mm -> Capacitor_SMD:C_1206_3216Metric_Pad1.33x1.80mm_HandSolder
- C6: renamed from C2; footprint Capacitor_THT:C_Disc_D6.0mm_W2.5mm_P5.00mm -> Capacitor_SMD:C_1206_3216Metric_Pad1.33x1.80mm_HandSolder
- C7: renamed from C3; footprint Capacitor_THT:C_Disc_D6.0mm_W2.5mm_P5.00mm -> Capacitor_SMD:C_1206_3216Metric_Pad1.33x1.80mm_HandSolder
- C8: renamed from C?; footprint Capacitor_THT:C_Disc_D3.8mm_W2.6mm_P2.50mm -> Capacitor_SMD:C_1206_3216Metric_Pad1.33x1.80mm_HandSolder
- C9: renamed from C46; footprint Capacitor_THT:C_Disc_D6.0mm_W2.5mm_P5.00mm -> Capacitor_SMD:C_1206_3216Metric_Pad1.33x1.80mm_HandSolder
- JP2, JP3: renamed from JP?; footprint (none) -> Jumper:SolderJumper-2_P1.3mm_Open_RoundedPad1.0x1.5mm
- R1: renamed from R12; footprint Resistor_THT:R_Axial_DIN0207_L6.3mm_D2.5mm_P7.62mm_Horizontal -> Resistor_SMD:R_1206_3216Metric_Pad1.30x1.75mm_HandSolder
- R10: renamed from R23; footprint Resistor_THT:R_Axial_DIN0207_L6.3mm_D2.5mm_P7.62mm_Horizontal -> Resistor_SMD:R_1206_3216Metric_Pad1.30x1.75mm_HandSolder
- R11: renamed from R24; footprint Resistor_THT:R_Axial_DIN0207_L6.3mm_D2.5mm_P7.62mm_Horizontal -> Resistor_SMD:R_1206_3216Metric_Pad1.30x1.75mm_HandSolder
- R12: renamed from R25; footprint Resistor_THT:R_Axial_DIN0207_L6.3mm_D2.5mm_P7.62mm_Horizontal -> Resistor_SMD:R_1206_3216Metric_Pad1.30x1.75mm_HandSolder
- R13: renamed from R26; footprint Resistor_THT:R_Axial_DIN0207_L6.3mm_D2.5mm_P7.62mm_Horizontal -> Resistor_SMD:R_1206_3216Metric_Pad1.30x1.75mm_HandSolder
- R14: renamed from R27; footprint Resistor_THT:R_Axial_DIN0207_L6.3mm_D2.5mm_P7.62mm_Horizontal -> Resistor_SMD:R_1206_3216Metric_Pad1.30x1.75mm_HandSolder
- R15, R3: renamed from R1; footprint Resistor_THT:R_Axial_DIN0207_L6.3mm_D2.5mm_P7.62mm_Horizontal -> Resistor_SMD:R_1206_3216Metric_Pad1.30x1.75mm_HandSolder
- R16: renamed from R28; footprint Resistor_THT:R_Axial_DIN0207_L6.3mm_D2.5mm_P7.62mm_Horizontal -> Resistor_SMD:R_1206_3216Metric_Pad1.30x1.75mm_HandSolder
- R17: renamed from R29; footprint Resistor_THT:R_Axial_DIN0207_L6.3mm_D2.5mm_P7.62mm_Horizontal -> Resistor_SMD:R_1206_3216Metric_Pad1.30x1.75mm_HandSolder
- R18: renamed from R5; footprint Resistor_THT:R_Axial_DIN0207_L6.3mm_D2.5mm_P7.62mm_Horizontal -> Resistor_SMD:R_1206_3216Metric_Pad1.30x1.75mm_HandSolder
- R19: renamed from R7; footprint Resistor_THT:R_Axial_DIN0207_L6.3mm_D2.5mm_P7.62mm_Horizontal -> Resistor_SMD:R_1206_3216Metric_Pad1.30x1.75mm_HandSolder
- R2: renamed from R13; footprint Resistor_THT:R_Axial_DIN0207_L6.3mm_D2.5mm_P7.62mm_Horizontal -> Resistor_SMD:R_1206_3216Metric_Pad1.30x1.75mm_HandSolder
- R20, R4: renamed from R2; footprint Resistor_THT:R_Axial_DIN0207_L6.3mm_D2.5mm_P7.62mm_Horizontal -> Resistor_SMD:R_1206_3216Metric_Pad1.30x1.75mm_HandSolder
- R21: renamed from R4; footprint Resistor_THT:R_Axial_DIN0207_L6.3mm_D2.5mm_P7.62mm_Horizontal -> Resistor_SMD:R_1206_3216Metric_Pad1.30x1.75mm_HandSolder
- R22: renamed from R6; footprint Resistor_THT:R_Axial_DIN0207_L6.3mm_D2.5mm_P7.62mm_Horizontal -> Resistor_SMD:R_1206_3216Metric_Pad1.30x1.75mm_HandSolder
- R23: renamed from R3; footprint Resistor_THT:R_Axial_DIN0207_L6.3mm_D2.5mm_P7.62mm_Horizontal -> Resistor_SMD:R_1206_3216Metric_Pad1.30x1.75mm_HandSolder
- R5: renamed from R30; footprint Resistor_THT:R_Axial_DIN0207_L6.3mm_D2.5mm_P7.62mm_Horizontal -> Resistor_SMD:R_1206_3216Metric_Pad1.30x1.75mm_HandSolder
- R6: renamed from R31; footprint Resistor_THT:R_Axial_DIN0207_L6.3mm_D2.5mm_P7.62mm_Horizontal -> Resistor_SMD:R_1206_3216Metric_Pad1.30x1.75mm_HandSolder
- R7: renamed from R32; footprint Resistor_THT:R_Axial_DIN0207_L6.3mm_D2.5mm_P7.62mm_Horizontal -> Resistor_SMD:R_1206_3216Metric_Pad1.30x1.75mm_HandSolder
- R8: renamed from R33; footprint Resistor_THT:R_Axial_DIN0207_L6.3mm_D2.5mm_P7.62mm_Horizontal -> Resistor_SMD:R_1206_3216Metric_Pad1.30x1.75mm_HandSolder
- R9: renamed from R22; footprint Resistor_THT:R_Axial_DIN0207_L6.3mm_D2.5mm_P7.62mm_Horizontal -> Resistor_SMD:R_1206_3216Metric_Pad1.30x1.75mm_HandSolder
- U1: renamed from U2; footprint (none) -> Package_SO:SOIC-14_3.9x8.7mm_P1.27mm
- gave numbers to parts that had none: 4
- renumbered C52 to C1, C15 to C11, C16 to C12, C50 to C2, C12 to C33, C13 to C34, C14 to C35, C36 to C38, C51 to C4, C43 to C41, C34 to C50, C35 to C51, C42 to C54, J11 to J1, J4 to J2, J5 to J3, J6 to J4, J3 to J5, J2 to J6, J8 to J7, J1 to J8, J7 to J9, L3 to L1, L1 to L2, L2 to L3, RN1 to RN2, U9 to U10, U5 to U2, U6 to U3, U3 to U5, U1 to U6, U7 to U9
Connections:
- net A10: no longer names the net of J1.52 (BA10)
- net A11: no longer names the net of J1.51 (BA11)
- net A12: no longer names the net of J1.50 (BA12)
- net A13: no longer names the net of J1.49 (BA13)
- net A14: no longer names the net of J1.48 (BA14)
- net A15: no longer names the net of J1.47 (BA15)
- net IRQ4: no longer names the net of J1.24 (IRQ4)
- no-connect marks 32 -> 39
